Commit message: fix: calibrate base_footprint grid height and prevent model duplication in gazebo

File: src/assem2_robot/urdf/Assem2.SLDASM.urdf (robot description, URDF)
Before this commit: robot assem2_robot, 6 links, 5 joints
Joints:
- joint base_footprint_joint: origin xyz=0 0 0 rpy=0 0 0 -> xyz=0.16662 0.10185 0.2269 rpy=0 0 0
- joint j1: origin xyz=0.139382908553347 -0.297269418402704 -0.146293994948754 rpy=2.33385883877157 0 0 -> xyz=0.13938 -0.29727 -0.14629 rpy=2.33386 0 0
- joint j2: origin xyz=0.139382908553346 0.0936811881755415 -0.147421263094464 rpy=2.56240825321655 0 0 -> xyz=0.13938 0.09368 -0.14742 rpy=2.56241 0 0
- joint j3: origin xyz=-0.472617091446653 -0.297269418402704 -0.146293994948754 rpy=-2.87166358324974 0 3.14159265358979 -> xyz=-0.47262 -0.29727 -0.14629 rpy=-2.87166 0 3.14159
- joint j4: origin xyz=-0.472617091446653 0.0934805663139231 -0.147799959833695 rpy=-1.29915826027407 0 3.14159265358979 -> xyz=-0.47262 0.09348 -0.14780 rpy=-1.29916 0 3.14159

Commit message: feat(perception): integrate 2D LiDAR, IMU, RGB-D camera and obstacle arena world

File: src/assem2_robot/urdf/Assem2.SLDASM.urdf (robot description, URDF)
Before this commit: robot assem2_robot, 6 links, 5 joints
Links:
- added link camera_link, mass 0.05; collision box size=0.025 0.09 0.025; visual box size=0.025 0.09 0.025
- added link camera_optical_frame
- added link imu_link, mass 0.01; visual box size=0.02 0.02 0.01
- added link lidar_link, mass 0.125; collision cylinder length=0.04 radius=0.04; visual cylinder length=0.04 radius=0.04
Joints:
- added joint camera_joint: type fixed, parent base_link, child camera_link, origin xyz=0.10 -0.10185 0.08 rpy=0 0 0
- added joint camera_optical_joint: type fixed, parent camera_link, child camera_optical_frame, origin xyz=0 0 0 rpy=-1.5707963 0 -1.5707963
- added joint imu_joint: type fixed, parent base_link, child imu_link, origin xyz=-0.16662 -0.10185 0.05 rpy=0 0 0
- added joint lidar_joint: type fixed, parent base_link, child lidar_link, origin xyz=-0.16662 -0.10185 0.13 rpy=0 0 0

Commit message: fix(kinematics): calibrate CAD-to-ROS coordinate frames, wheel axes, and skid-steer friction

File: src/assem2_robot/urdf/Assem2.SLDASM.urdf (robot description, URDF)
Before this commit: robot assem2_robot, 10 links, 9 joints
Joints:
- joint base_footprint_joint: origin xyz=0.16662 0.10185 0.2269 rpy=0 0 0 -> xyz=0.10185 -0.16662 0.2269 rpy=0 0 -1.5707963
- joint camera_joint: origin xyz=0.10 -0.10185 0.08 rpy=0 0 0 -> xyz=-0.16662 0.15 0.08 rpy=0 0 1.5707963
- joint imu_joint: origin xyz=-0.16662 -0.10185 0.05 rpy=0 0 0 -> xyz=-0.16662 -0.10185 0.05 rpy=0 0 1.5707963
- joint j1: axis 1 0 0 -> -1 0 0
- joint j2: axis 1 0 0 -> -1 0 0
- joint lidar_joint: origin xyz=-0.16662 -0.10185 0.13 rpy=0 0 0 -> xyz=-0.16662 -0.10185 0.133 rpy=0 0 1.5707963

Commit message: fix(physics): lower chassis center-of-mass and use cylinder wheel collision primitives to prevent tipping

File: src/assem2_robot/urdf/Assem2.SLDASM.urdf (robot description, URDF)
Before this commit: robot assem2_robot, 10 links, 9 joints
Links:
- link base_link: mass 20.0 -> 22.0
- link w1: mass 1.1928 -> 1.5; geometry collision cylinder length=0.06 radius=0.08; visual mesh filename=package://assem2_robot/meshes/w1.STL
- link w2: mass 1.1928 -> 1.5; geometry collision cylinder length=0.06 radius=0.08; visual mesh filename=package://assem2_robot/meshes/w2.STL
- link w3: mass 1.1928 -> 1.5; geometry collision cylinder length=0.06 radius=0.08; visual mesh filename=package://assem2_robot/meshes/w3.STL
- link w4: mass 1.1928 -> 1.5; geometry collision cylinder length=0.06 radius=0.08; visual mesh filename=package://assem2_robot/meshes/w4.STL
Joints:
- joint j1: limit effort=100 velocity=100 -> effort=40 velocity=25
- joint j2: limit effort=100 velocity=100 -> effort=40 velocity=25
- joint j3: limit effort=100 velocity=100 -> effort=40 velocity=25
- joint j4: limit effort=100 velocity=100 -> effort=40 velocity=25

Commit message: fix(kinematics): invert wheel rotation axes so positive teleop velocity drives robot forward

File: src/assem2_robot/urdf/Assem2.SLDASM.urdf (robot description, URDF)
Before this commit: robot assem2_robot, 10 links, 9 joints
Joints:
- joint j1: axis -1 0 0 -> 1 0 0
- joint j2: axis -1 0 0 -> 1 0 0
- joint j3: axis 1 0 0 -> -1 0 0
- joint j4: axis 1 0 0 -> -1 0 0

Commit message: feat(sensors): enhance sensor mounting risers, optical frame alignment, and visual aesthetics

File: src/assem2_robot/urdf/Assem2.SLDASM.urdf (robot description, URDF)
Before this commit: robot assem2_robot, 10 links, 9 joints
Links:
- added link camera_mount_link, mass 0.04; visual box size=0.03 0.08 0.01
- added link lidar_mount_link, mass 0.08; collision cylinder length=0.03 radius=0.045; visual cylinder length=0.03 radius=0.045
- link camera_link: mass 0.05 -> 0.07; geometry collision box size=0.025 0.09 0.025; visual box size=0.025 0.09 0.025
- link imu_link: geometry visual box size=0.025 0.025 0.01
- link lidar_link: geometry collision cylinder length=0.04 radius=0.04; visual cylinder length=0.015 radius=0.035
Joints:
- added joint camera_mount_joint: type fixed, parent base_link, child camera_mount_link, origin xyz=-0.16662 0.15 0.065 rpy=0 0 1.5707963
- added joint lidar_mount_joint: type fixed, parent base_link, child lidar_mount_link, origin xyz=-0.16662 -0.10185 0.105 rpy=0 0 1.5707963
- joint camera_joint: origin xyz=-0.16662 0.15 0.08 rpy=0 0 1.5707963 -> xyz=0 0 0.01 rpy=0 0 0; parent base_link -> camera_mount_link
- joint camera_optical_joint: origin xyz=0 0 0 rpy=-1.5707963 0 -1.5707963 -> xyz=0.013 0 0.0125 rpy=-1.5707963 0 -1.5707963
- joint imu_joint: origin xyz=-0.16662 -0.10185 0.05 rpy=0 0 1.5707963 -> xyz=-0.16662 -0.10185 0.02 rpy=0 0 1.5707963
- joint lidar_joint: origin xyz=-0.16662 -0.10185 0.133 rpy=0 0 1.5707963 -> xyz=0 0 0.03 rpy=0 0 0; parent base_link -> lidar_mount_link

Commit message: fix(chassis): align physical front bumper with driving forward heading and mount camera on front bumper

File: src/assem2_robot/urdf/Assem2.SLDASM.urdf (robot description, URDF)
Before this commit: robot assem2_robot, 12 links, 11 joints
Joints:
- joint base_footprint_joint: origin xyz=0.10185 -0.16662 0.2269 rpy=0 0 -1.5707963 -> xyz=-0.10185 0.16662 0.2269 rpy=0 0 1.5707963
- joint camera_mount_joint: origin xyz=-0.16662 0.15 0.065 rpy=0 0 1.5707963 -> xyz=-0.16662 -0.355 0.065 rpy=0 0 -1.5707963
- joint imu_joint: origin xyz=-0.16662 -0.10185 0.02 rpy=0 0 1.5707963 -> xyz=-0.16662 -0.10185 0.02 rpy=0 0 -1.5707963
- joint j1: axis 1 0 0 -> -1 0 0
- joint j2: axis 1 0 0 -> -1 0 0
- joint j3: axis -1 0 0 -> 1 0 0
- joint j4: axis -1 0 0 -> 1 0 0
- joint lidar_mount_joint: origin xyz=-0.16662 -0.10185 0.105 rpy=0 0 1.5707963 -> xyz=-0.16662 -0.10185 0.105 rpy=0 0 -1.5707963

Commit message: feat(civil): add Civil Architectural simulation, 2D SLAM mapping, and smooth teleoperation
- Add civil floor simulation world (civil_world.sdf) and launcher (civil_simulation.launch.py)
- Enable RobotModel in civil_display.rviz and display.rviz
- Fix civil_teleop.py: continuous cruise drive mode by default, robust multi-byte arrow key parsing, and remove premature quit on 'Q'
- Add convenience launchers: run_civil_mapping.sh, run_teleop.sh, run_civil_nav.sh, and save_civil_map.sh
- Include 2D SLAM occupancy grid civil maps and engineering documentation
- Document civil simulation and teleop execution commands in README.md, COMMANDS.md, and CHEAT_SHEET.md

File: src/assem2_robot/urdf/Assem2.SLDASM.urdf (robot description, URDF)
Before this commit: robot assem2_robot, 12 links, 11 joints
Links:
- link base_link: geometry collision box size=0.48 0.32 0.16; visual mesh filename=package://assem2_robot/meshes/base_link.STL
